Commit message: local planner pkg added
The local planner pkg will recive the hovex hull caluction of each clouster to cevert it into 2d and i will calculate if there is a obstacle and if the robot can create a obstacle obvoidance action

File: sdv_robot_description/urdf/robot.urdf (robot description, URDF)
Before this commit: robot dasautonomeauto, 2 links, 1 joints
Links:
- removed link velodyne
Joints:
- removed joint velodyne_base_mount_joint

Commit message: lidar clouster convex hull addded
Lidar convex hull added to create a grid

File: sdv_robot_description/urdf/robot.urdf (robot description, URDF)
Before this commit: robot dasautonomeauto, 1 links, 0 joints
Links:
- added link base_footprint
- added link detector_wall
Joints:
- added joint base_link_joint: type fixed, parent chassis_link, child base_footprint, origin xyz=0 0 0.5 rpy=0 0 0
- added joint detector_wall_joint: type fixed, parent chassis_link, child detector_wall, origin xyz=0 1.45 1.1 rpy=0 0 0

Commit message: readme updated

File: sdv_robot_description/urdf/robot.urdf (robot description, URDF)
Before this commit: robot dasautonomeauto, 3 links, 2 joints
Links:
- added link velodyne
- link chassis_link: mass 125.0 -> None; geometry visual mesh filename=file://$(find sdv_robot_description)/meshes/hooke.dae scale=0.001 0.001 0.001
Joints:
- added joint velodyne_base_mount_joint: type fixed, parent chassis_link, child velodyne, origin xyz=0 0 1.8 rpy=-0.174533 0 0
- joint base_link_joint: origin xyz=0 0 0.5 rpy=0 0 0 -> xyz=0 0 -0.1 rpy=0 0 0
- joint detector_wall_joint: origin xyz=0 1.45 1.1 rpy=0 0 0 -> xyz=0 1 0 rpy=0 0 0
