Commit message: waypoints and urdf fixed

File: sdv_robot_description/urdf/Autoreifen.xacro (robot description, xacro)
@@ -1,9 +1,5 @@
 <?xml version="1.0"?>
-<robot name="sdv_car" xmlns:xacro="http://www.ros.org/wiki/xacro">
-<!--
-  <xacro:property name="tire_dia" value="0.750"/>
-  <xacro:property name="tire_width" value="0.125"/>
-  <xacro:property name="hub_dia" value="0.235"/>   -->
-  <xacro:property name="tire_dia" value="0.750"/>  <!-- Reduced from 0.440 -->
+<robot name="dasautonomeauto" xmlns:xacro="http://www.ros.org/wiki/xacro">
+  <xacro:property name="tire_dia" value="0.350"/>  <!-- Reduced from 0.440 -->
   <xacro:property name="tire_width" value="0.195"/>  <!-- Reduced from 0.195 -->
   <xacro:property name="hub_dia" value="0.235"/>  <!-- Reduced from 0.235 -->
@@ -16,10 +12,10 @@
   <xacro:property name="axle_vel_limit" value="39.02"/>
   <!-- Properties of the car -->
-  <xacro:property name="front_wheel_x" value="0.087346576344423"/>
-  <xacro:property name="front_wheel_y" value="0.695625727164768"/>
-  <xacro:property name="front_wheel_z" value="0.2594929592556163"/>
-  <xacro:property name="rear_wheel_x" value="-2.04780116842239"/>
-  <xacro:property name="rear_wheel_y" value="0.695625727164768"/>
-  <xacro:property name="rear_wheel_z" value="0.2594929592556163"/>
+  <xacro:property name="front_wheel_x" value="0.787346576344423"/>
+  <xacro:property name="front_wheel_y" value="0.495625727164768"/>
+  <xacro:property name="front_wheel_z" value="0.1094929592556163"/>
+  <xacro:property name="rear_wheel_x" value="1.04780116842239"/>
+  <xacro:property name="rear_wheel_y" value="0.495625727164768"/>
+  <xacro:property name="rear_wheel_z" value="0.1094929592556163"/>
   <!-- Degree-to-radian conversions -->
   <xacro:property name="degrees_45" value="0.785398163"/>
@@ -29,5 +25,5 @@
   <xacro:property name="servo_no_load_speed" value="25"/> <!-- check -->
   <material name="black">
-      <color rgba="0 0 0 1"/>
+      <color rgba="1.0 1.0 1.0 1.0"/>
   </material>
   <xacro:macro name="thick_walled_tube_inertial"
@@ -61,5 +57,5 @@
     <joint name="${lr_prefix}_steering_joint" type="revolute">
       <origin xyz="${fr_reflect * front_wheel_x} ${lr_reflect * front_wheel_y} ${-front_wheel_z}" rpy="0 ${degrees_90} 0"/>
-      <parent link="base_link"/>
+      <parent link="chassis_link"/>
       <child link="${lr_prefix}_steering_link"/>
       <axis xyz="-1 0 0"/>
@@ -125,5 +121,5 @@
     </link>
     <joint name="${lr_prefix}_${fr_prefix}_axle" type="continuous">
-      <parent link="base_link"/>
+      <parent link="chassis_link"/>
       <child link="${lr_prefix}_${fr_prefix}_wheel"/>
       <origin xyz="${fr_reflect * rear_wheel_x} ${lr_reflect * rear_wheel_y} ${-rear_wheel_z}" rpy="1.5708 0 0"/>

File: sdv_robot_description/urdf/zf_car.urdf (robot description, URDF)
Before this commit: robot dasautonomeauto, 3 links, 2 joints
Links:
- added link warning_obstacle
- link chassis_link: mass 125.0 -> None; geometry visual mesh filename=file://$(find sdv_robot_description)/meshes/sdv.stl
Joints:
- added joint warning_base_mount_joint: type fixed, parent chassis_link, child warning_obstacle, origin xyz=1.2 0.0 0.0 rpy=0 0 0
- joint base_link_joint: child chassis_link -> base_footprint; origin xyz=0 0 0.5 rpy=0 0 0 -> xyz=0 0 -0.1 rpy=0 0 0; parent base_footprint -> chassis_link
