Commit message: data

File: sdv_robot_description/urdf/test_lidar_camara.urdf (robot description, URDF)
Before this commit: robot dasautonomeauto, 6 links, 5 joints
Links:
- removed link base_footprint
- removed link rslidar
- removed link warning_obstacle
- link chassis_link: geometry 
Joints:
- removed joint base_link_joint
- removed joint rslidar_base_mount_joint
- removed joint warning_base_mount_joint
- joint default_cam_base_mount_joint: origin xyz=0.05 0 1.18 rpy=0 0 0 -> xyz=0.05 0 0.75 rpy=0 0 0
- joint velodyne_base_mount_joint: origin xyz=0 0 1.23 rpy=0 0 0 -> xyz=0 0 0.8 rpy=0 0 0
