Commit message: vector of obstacles added in oder to called in the franet pkg

File: sdv_robot_description/urdf/hook.urdf (robot description, URDF)
Before this commit: robot dasautonomeauto, 3 links, 2 joints
Links:
- added link warning_obstacle
Joints:
- added joint warning_base_mount_joint: type fixed, parent chassis_link, child warning_obstacle, origin xyz=1.2 0.0 0.0 rpy=0 0 0

Commit message: franet frame added

File: sdv_robot_description/urdf/hook.urdf (robot description, URDF)
Before this commit: robot dasautonomeauto, 4 links, 3 joints
Links:
- link chassis_link: geometry visual mesh filename=file://$(find sdv_robot_description)/meshes/hook_pix.stl scale=0.001 0.001 0.001

Commit message: frenet updated

File: sdv_robot_description/urdf/hook.urdf (robot description, URDF)
Before this commit: robot dasautonomeauto, 4 links, 3 joints
Links:
- removed link rslidar
- added link velodyne
Joints:
- joint base_link_joint: origin xyz=0 0 -0.1 rpy=0 0 0 -> xyz=0 0 -0.38 rpy=0 0 0
- joint rslidar_base_mount_joint: child rslidar -> velodyne; origin xyz=0 0 1.2 rpy=0 0 0 -> xyz=0 0 1.23 rpy=0 0 0

Commit message: frenet update

File: sdv_robot_description/urdf/hook.urdf (robot description, URDF)
Before this commit: robot dasautonomeauto, 4 links, 3 joints
Links:
- added link rslidar
Joints:
- added joint velodyne_base_mount_joint: type fixed, parent chassis_link, child velodyne, origin xyz=0 0 1.23 rpy=0 0 0
- joint rslidar_base_mount_joint: child velodyne -> rslidar

Commit message: lidar trking added

File: sdv_robot_description/urdf/hook.urdf (robot description, URDF)
Before this commit: robot dasautonomeauto, 5 links, 4 joints
Links:
- link rslidar: geometry visual cylinder length=0.073 radius=0.04

Commit message: plane_getter updated

File: sdv_robot_description/urdf/hook.urdf (robot description, URDF)
Before this commit: robot dasautonomeauto, 6 links, 5 joints
Links:
- link chassis_link: geometry visual mesh filename=file://$(find sdv_robot_description)/meshes/sdv.stl
- link rslidar: geometry 
- link velodyne: geometry visual cylinder length=0.073 radius=0.04
Joints:
- joint rslidar_base_mount_joint: origin xyz=0 0 1.23 rpy=0 0 0 -> xyz=0 0 1.8 rpy=0 0 0
- joint velodyne_base_mount_joint: origin xyz=0 0 1.23 rpy=0 0 0 -> xyz=0 0 1.8 rpy=0 0.174533 0

Commit message: oppinal plannet modification

File: sdv_robot_description/urdf/hook.urdf (robot description, URDF)
Before this commit: robot dasautonomeauto, 6 links, 5 joints
Links:
- link chassis_link: geometry visual mesh filename=file://$(find sdv_robot_description)/meshes/hook_pix.stl scale=0.001 0.001 0.001
Joints:
- joint rslidar_base_mount_joint: origin xyz=0 0 1.8 rpy=0 0 0 -> xyz=0 0 1.23 rpy=0 0 0
- joint velodyne_base_mount_joint: origin xyz=0 0 1.8 rpy=0 0.174533 0 -> xyz=0 0 1.23 rpy=0 0 0

Commit message: tf working fine

File: sdv_robot_description/urdf/hook.urdf (robot description, URDF)
Before this commit: robot dasautonomeauto, 6 links, 5 joints
Links:
- removed link chassis_link
- removed link default_cam
- added link base_link; visual mesh filename=file://$(find sdv_robot_description)/meshes/sdv.stl
Joints:
- removed joint default_cam_base_mount_joint
- joint base_link_joint: parent chassis_link -> base_link
- joint rslidar_base_mount_joint: parent chassis_link -> base_link
- joint velodyne_base_mount_joint: origin xyz=0 0 1.23 rpy=0 0 0 -> xyz=0 0 1.8 rpy=0 0.174533 0; parent chassis_link -> base_link
- joint warning_base_mount_joint: parent chassis_link -> base_link

File: sdv_robot_description/urdf/zf_car.urdf (robot description, URDF)
Before this commit: robot dasautonomeauto, 4 links, 3 joints
Links:
- link chassis_link: mass None -> 125.0; geometry collision mesh filename=file://$(find sdv_robot_description)/meshes/sdv.stl; visual mesh filename=file://$(find sdv_robot_description)/meshes/sdv.stl
Joints:
- joint base_link_joint: child base_footprint -> chassis_link; origin xyz=0 0 -0.1 rpy=0 0 0 -> xyz=0 0 0.5 rpy=0 0 0; parent chassis_link -> base_footprint
