Commit message: robot des

File: sdv_robot_description/urdf/golf_car.urdf (robot description, URDF)
Before this commit: robot dasautonomeauto, 4 links, 3 joints
Links:
- added link velodyne; visual cylinder length=0.073 radius=0.04
Joints:
- added joint velodyne_base_mount_joint: type fixed, parent chassis_link, child velodyne, origin xyz=0 0 1.6 rpy=0 0 0

File: sdv_robot_description/urdf/hook.urdf (robot description, URDF)
Before this commit: robot dasautonomeauto, 5 links, 4 joints
Links:
- link base_link: geometry visual mesh filename=file://$(find sdv_robot_description)/meshes/hook_pix.stl scale=0.001 0.001 0.001
Joints:
- joint velodyne_base_mount_joint: origin xyz=0 0 1.8 rpy=0 0.174533 0 -> xyz=0 0 1.8 rpy=0 0 0

File: sdv_robot_description/urdf/zf_car.urdf (robot description, URDF)
Before this commit: robot dasautonomeauto, 4 links, 3 joints
Links:
- removed link base_footprint
- removed link chassis_link
- removed link velodyne
- removed link warning_obstacle
- added link base_link; visual mesh filename=file://$(find sdv_robot_description)/meshes/sdv.stl
Joints:
- removed joint base_link_joint
- removed joint velodyne_base_mount_joint
- removed joint warning_base_mount_joint
